File: hardware/pcb/xiao-rv01β/xiao-rv01β.kicad_sch (KiCad schematic)
At the start: 34 parts, among them J1 Conn_01x02_Pin, J2 Conn_01x02_Pin, J3 Conn_01x02_Pin, J4 Conn_01x02_Pin, J5 Conn_01x02_Socket, M1 DC_Motor_3V, M2 DC_Motor_3V, Q1 P-Ch -20V/-3A, U1 DRV8835, U2 XIAO ESP32C6

Commit message: completed the 1st edit of xiao-rv01β
Signed-off-by: Takuto Nagami <logica0419@gmail.com>
Parts:
- removed D2, D3: SBD 45V/2A, Diode_THT:D_DO-41_SOD81_P10.16mm_Horizontal, symbol Diode:SB5H90
- removed J3: Conn_01x02_Pin, Connector_JST:JST_XH_B2B-XH-A_1x02_P2.50mm_Vertical, symbol Connector:Conn_01x02_Pin
- added BZ1: Buzzer, sglib:buzzer 5.5mm, symbol Device:Buzzer
- added C2, C8, C9: 0.1μF, symbol Device:C
- added J3, J5: Conn_01x02_Socket, symbol Connector:Conn_01x02_Socket
- added J7: Conn_01x10_Pin, symbol Connector:Conn_01x10_Pin
- added J8: Conn_02x10_Pin, symbol Connector_Generic:Conn_02x10_Top_Bottom
- added J9: Conn_01x04_Pin, symbol Connector:Conn_01x04_Pin
- added LED1, LED2, LED3, LED4, LED5, LED6: SK6812MINI, foostan/kbd:YS-SK6812MINI-E, symbol foostan/kbd:YS-SK6812MINI-E
- added LED7: Green, symbol Device:LED
- added LED8: Orange, symbol Device:LED
- added R1, R2, R3, R4: 100Ω, symbol Device:R
- added R10, R7, R8, R9: 4.7kΩ, symbol Device:R
- added R17, R19: 1kΩ, Resistor_THT:R_Axial_DIN0207_L6.3mm_D2.5mm_P7.62mm_Horizontal, symbol Device:R
- added R18: 2.2kΩ, Resistor_THT:R_Axial_DIN0207_L6.3mm_D2.5mm_P7.62mm_Horizontal, symbol Device:R
- added SEN1, SEN2, SEN3, SEN4: LBR-123F, OptoDevice:Vishay_CNY70, symbol Sensor_Proximity:CNY70
- added SEN5: HC-SR04, symbol HC-SR04:HC-SR04
- added SW1, SW2, SW3, SW4, SW5: SW_Push, symbol Switch:SW_Push
- added U2, U4: ADS1015, Package_SO:TSSOP-10_3x3mm_P0.5mm, symbol Analog_ADC:ADS1015IDGS
- added U5: MCP23017, Package_DIP:DIP-28_W7.62mm, symbol Interface_Expansion:MCP23017x-x-SP
- J2: renamed from J5; now not fitted
- M1, M2: now not fitted
- Q1: value P-Ch -20V/-3A -> P-Ch -12V/-6A
- R14: renamed from R8; value 22kΩ -> 33kΩ
- R15: renamed from R4; value 100kΩ -> 33kΩ
- U1: renamed from U2; footprint Seeed_Studio_XIAO_Series:XIAO-ESP32-C6-SMD -> New_XIAO_Series_Footprints:XIAO-ESP32-C3-DIP-SMD
- U3: renamed from U1; symbol drv8835:DRV8835DSSR -> DRV8835:DRV8835DSSR
- renumbered C3 to C1, C1 to C3, C6 to C4, C4 to C5, C5 to C6, C2 to C7, J4 to J1, J1 to J4, J2 to J6, R7 to R11, R1 to R12, R2 to R13, R6 to R16, R3 to R5, R5 to R6
Connections:
- net 3V3: now also U1.12 (3V3), C2.1, C8.2, C9.2, J8.1 (Pin_1), J8.10 (Pin_10), J8.2 (Pin_2), J8.3 (Pin_3), J8.4 (Pin_4), J8.5 (Pin_5), J8.6 (Pin_6), J8.7 (Pin_7), J8.8 (Pin_8), J8.9 (Pin_9), J9.3 (Pin_3), LED1.1 (VDD), LED2.1 (VDD), LED3.1 (VDD), LED4.1 (VDD), LED5.1 (VDD), LED6.1 (VDD), LED7.2 (A), R1.1, R2.1, R3.1, R4.1, SEN1.3 (C), SEN2.3 (C), SEN3.3 (C), SEN4.3 (C), SEN5.1 (Vcc), U2.1 (ADDR), U2.8 (VDD), U4.8 (VDD), U5.18 (~{RESET}), U5.9 (V_{DD})
- net GND: now also BT1.2 (-), BZ1.2 (-), C2.2, C8.1, C9.1, J8.11 (Pin_11), J8.12 (Pin_12), J8.13 (Pin_13), J8.14 (Pin_14), J8.15 (Pin_15), J8.16 (Pin_16), J8.17 (Pin_17), J8.18 (Pin_18), J8.19 (Pin_19), J8.20 (Pin_20), J9.4 (Pin_4), LED1.3 (VSS), LED2.3 (VSS), LED3.3 (VSS), LED4.3 (VSS), LED5.3 (VSS), LED6.3 (VSS), R10.2, R17.1, R18.1, R7.2, R8.2, R9.2, SEN1.2 (K), SEN2.2 (K), SEN3.2 (K), SEN4.2 (K), SEN5.4 (GND), SW1.2, SW2.2, SW3.2, SW4.2, SW5.2, U2.3 (GND), U4.1 (ADDR), U4.3 (GND), U5.10 (V_{SS}), U5.15 (A0), U5.16 (A1), U5.17 (A2)
- net MD_APHASE: now also U5.27 (GPA6)
- net MD_BPHASE: now also U5.28 (GPA7)
- net NEO_PIXEL: now also LED1.4 (DIN)
- net SCL: now also J9.1 (Pin_1), U2.10 (SCL), U4.10 (SCL), U5.13 (SDA)
- net SDA: now also J9.2 (Pin_2), U2.9 (SDA), U4.9 (SDA), U5.12 (SCK)
- net VBUS: now also U1.14 (VBUS), LED8.2 (A)
- net at F1.1: now also BT1.1 (+)
- net at M1.1 (+): now also J3.1 (Pin_1)
- net at M1.2 (-): now also J3.2 (Pin_2)
- net at M2.1 (+): now also J5.1 (Pin_1)
- net at M2.2 (-): now also J5.2 (Pin_2)
- net EXT_ADC/PWM1 renamed EXT1_ADC/PWM
- net EXT1_ADC/PWM: now also J7.1 (Pin_1)
- net EXT_ADC/PWM2 renamed EXT2_ADC/PWM
- net EXT2_ADC/PWM: now also J7.2 (Pin_2)
- net EXT_PWM1 renamed EXT3_PWM
- net EXT3_PWM: now also J7.3 (Pin_3)
- net EXT_PWM2 renamed BUZZER
- net BUZZER: now also R19.2
- new net: SEN5.2 (Trigger), U5.1 (GPB0)
- new net: SEN5.3 (Echo), U5.2 (GPB1)
- new net: SW1.1, U5.3 (GPB2)
- new net: SW2.1, U5.4 (GPB3)
- new net: SW3.1, U5.5 (GPB4)
- new net: SW4.1, U5.6 (GPB5)
- new net: SW5.1, U5.7 (GPB6)
- new net: R4.2, SEN4.1 (A)
- new net: R10.1, SEN4.4 (E), U2.4 (AIN0)
- new net: R3.2, SEN3.1 (A)
- new net: R9.1, SEN3.4 (E), U2.5 (AIN1)
- new net: LED3.2 (DOUT), LED5.4 (DIN)
- new net: LED1.2 (DOUT), LED3.4 (DIN)
- new net: LED8.1 (K), R18.2
- new net: LED7.1 (K), R17.2
- new net: BZ1.1 (+), R19.1
- new net: LED4.2 (DOUT), LED6.4 (DIN)
- new net: LED2.4 (DIN), LED5.2 (DOUT)
- new net: LED2.2 (DOUT), LED4.4 (DIN)
- new net: R2.2, SEN2.1 (A)
- new net: R8.1, SEN2.4 (E), U2.6 (AIN2)
- new net: R1.2, SEN1.1 (A)
- new net: R7.1, SEN1.4 (E), U2.7 (AIN3)
- new net EXT10_GPIO: J7.10 (Pin_10), U5.23 (GPA2)
- new net EXT4_ADC: J7.4 (Pin_4), U4.4 (AIN0)
- new net EXT5_ADC: J7.5 (Pin_5), U4.5 (AIN1)
- new net EXT6_ADC: J7.6 (Pin_6), U4.6 (AIN2)
- new net EXT7_ADC: J7.7 (Pin_7), U4.7 (AIN3)
- new net EXT8_GPIO: J7.8 (Pin_8), U5.21 (GPA0)
- new net EXT9_GPIO: J7.9 (Pin_9), U5.22 (GPA1)
- no-connect marks 8 -> 17
Other:
- note added: "ADC #1 & Reflective Sensors"
- note added: "ADC #2"
- note added: "Buzzer"
- note added: "Extention Pins"
- note added: "I/O Expander & Sensors"
- note added: "LEDs"
- note added: "Motor Driver"
- note added: "OLED Display"
- note added: "Power & MCU"
- company: (none) -> TinyGo Keeb
- title: (none) -> xiao-rv01β
- moved on the sheet: C1, C3, C4, C5, C6, C7, D1, F1, FB1, FB2, FB3, FB4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

Commit message: add power switch & organize
Signed-off-by: Takuto Nagami <logica0419@gmail.com>
Parts:
- added Q2: P-Ch -12V/-6A, Package_TO_SOT_THT:TO-251-3_Vertical, symbol Transistor_FET:Q_PMOS_GDS
- added R20: 100kΩ, Resistor_THT:R_Axial_DIN0207_L6.3mm_D2.5mm_P10.16mm_Horizontal, symbol Device:R
- added SW6: SW_SPDT, symbol Switch:SW_SPDT
Connections:
- net GND: now also SW6.1 (A)
- net at D1.1 (K), J1.1 (Pin_1), Q1.3 (S)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: now also Q2.2 (D); no longer F1.2
- new net: F1.2, Q2.3 (S), R20.1
- new net: Q2.1 (G), R20.2, SW6.2 (B)
- no-connect marks 17 -> 18
Other:
- moved on the sheet: BT1, C1, C2, C3, C4, C5, C6, C7, C8, C9, D1, F1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
