File: hardware/pcb/xiao-rv01β/xiao-rv01β.kicad_sch (KiCad schematic)
At the start: 75 parts, among them J1 Conn_01x02_Pin, J2 Conn_01x02_Socket, J3 Conn_01x02_Socket, J4 Conn_01x02_Pin, J5 Conn_01x02_Socket, J6 Conn_01x02_Pin, J7 Conn_01x10_Pin, J8 Conn_02x10_Pin, J9 Conn_01x04_Pin, M1 DC_Motor_3V, M2 DC_Motor_3V, Q1 P-Ch -12V/-6A, Q2 P-Ch -12V/-6A, SW1 SW_Push, SW2 SW_Push, SW3 SW_Push, SW4 SW_Push, SW5 SW_Push, SW6 SW_SPDT, U1 XIAO ESP32C6, U2 ADS1015, U3 DRV8835, U4 ADS1015, U5 MCP23017

Commit message: modified distance sensor & tweaks
Signed-off-by: Takuto Nagami <logica0419@gmail.com>
Parts:
- removed C4: 100μF/10V, symbol Device:C_Polarized
- removed LED5, LED6: SK6812MINI, foostan/kbd:YS-SK6812MINI-E, symbol foostan/kbd:YS-SK6812MINI-E
- removed SEN5: HC-SR04, symbol HC-SR04:HC-SR04
- added C10, C4: 47µF/10V, symbol Device:C
- added SEN5: GP2Y0E03, symbol GP2Y0E03:GP2Y0E03
- U1: footprint New_XIAO_Series_Footprints:XIAO-ESP32-C3-DIP-SMD -> New_XIAO_Series_Footprints:XIAO-ESP32-C6-DIP
- renumbered C8 to C7, C9 to C8, C7 to C9, J9 to J7, J7 to J8, J8 to J9, LED7 to LED5, LED8 to LED6, R7 to R10, R8 to R11, R9 to R12, R10 to R13, R11 to R14, R20 to R15, R14 to R16, R16 to R17, R19 to R18, R17 to R19, R18 to R20, R12 to R6, R15 to R7, R13 to R8, R6 to R9, SW6 to SW1, SW1 to SW2, SW2 to SW3, SW3 to SW4, SW4 to SW5, SW5 to SW6, U4 to U3, U3 to U4
Connections:
- net 3V3: now also C10.2, SEN5.1 (VDD), SEN5.4 (VIN_IO), SEN5.5 (GPIO1)
- net GND: now also C10.1, C4.1, SEN5.3 (GND)
- net MD_APHASE: now also U5.7 (GPB6); no longer U5.27 (GPA6)
- net MD_BPHASE: now also U5.8 (GPB7); no longer U5.28 (GPA7)
- net SCL: now also SEN5.6 (SCL)
- net SDA: now also SEN5.7 (SDA)
- net VM: now also C4.2
- net at U5.1 (GPB0): now also SW2.1
- net at U5.2 (GPB1): now also SW3.1
- net at U5.3 (GPB2): now also SW4.1; no longer SW2.1
- net at U5.4 (GPB3): now also SW5.1; no longer SW3.1
- net at U5.5 (GPB4): now also SW6.1; no longer SW4.1
- net at U5.6 (GPB5): no longer SW5.1
- net at LED3.2 (DOUT): now also LED2.4 (DIN)
- no-connect marks 18 -> 21
Other:
- note added: "Distance Sensor"
- note added: "I/O Expander & Switches"
- note removed: "I/O Expander & Sensors"
- moved on the sheet: BZ1, C2, C3, C5, C6, C7, C8, C9, FB1, FB2, FB3, FB4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
